File: pcb/bike-dash/control-board.brd (EAGLE design)
At the start: 86 x 50 mm, 29 parts, among them IC1_3V3 LM2575S, IC1_L9637D L9637D, IC2_5V LM2575S

Commit message: changes to pcb
Routing:
- net GND: track 294.5 -> 302.2 mm
Changed lines of the file:
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@@
 <wire x1="38.0502" y1="24.88" x2="38.185878125" y2="24.744321875" width="0.1524" layer="1"/>
 <wire x1="40.2336" y1="18.1356" x2="40.26" y2="18" width="0.1524" layer="1"/>
-<wire x1="41.6052" y1="25.4508" x2="48.1584" y2="25.4508" width="0.1524" layer="1"/>
-<wire x1="48.1584" y1="25.4508" x2="48.265" y2="25.54" width="0.1524" layer="1"/>
-<wire x1="41.6052" y1="25.4508" x2="40.743475" y2="24.88" width="0.1524" layer="1"/>
-<wire x1="38.0502" y1="24.88" x2="40.743475" y2="24.88" width="0.1524" layer="1"/>
+<wire x1="48.265" y1="25.54" x2="43.265" y2="25.54" width="0.1524" layer="1"/>
+<wire x1="43.265" y1="25.54" x2="42.3542" y2="26.4508" width="0.1524" layer="1"/>
+<wire x1="42.3542" y1="26.4508" x2="34.621" y2="26.4508" width="0.1524" layer="1"/>
+<wire x1="38.0502" y1="24.88" x2="36.1918" y2="24.88" width="0.1524" layer="1"/>
+<wire x1="36.1918" y1="24.88" x2="34.621" y2="26.4508" width="0.1524" layer="1"/>
 <wire x1="29.2608" y1="23.9268" x2="26.3652" y2="26.8224" width="0.1524" layer="1"/>
 <wire x1="35.577584375" y1="23.9268" x2="29.2608" y2="23.9268" width="0.1524" layer="1"/>
